Commit message: Add hardware parameters

File: clearpath_manipulators_description/urdf/lift/ewellix.urdf.xacro (robot description, xacro)
@@ -17,4 +17,10 @@
     use_fake_hardware:=''
     sim_ignition:=''
+    port=''
+    baud=''
+    timeout=''
+    conversion=''
+    rated_effort=''
+    tolerance=''
     ">
     <!-- Default Description Parameters -->
@@ -27,4 +33,11 @@
     <xacro:property name="_use_fake_hardware" value="false" />
     <xacro:property name="_sim_ignition" value="$(arg is_sim)" />
+    <!-- Default Hardware Parameters -->
+    <xacro:property name="_port" value="/dev/ttyUSB0"/>
+    <xacro:property name="_baud" value="38400"/>
+    <xacro:property name="_timeout" value="1000"/>
+    <xacro:property name="_conversion" value="3200"/>
+    <xacro:property name="_rated_effort" value="2000"/>
+    <xacro:property name="_tolerance" value="0.005"/>
     <!-- Parameter Overwrites -->
     <xacro:if value="${initial_positions != ''}"> <xacro:property name="_initial_positions" value="${initial_positions}" lazy_eval="false"/> </xacro:if>
@@ -35,4 +48,10 @@
     <xacro:if value="${use_fake_hardware != ''}"> <xacro:property name="_use_fake_hardware" value="${use_fake_hardware}" lazy_eval="false"/> </xacro:if>
     <xacro:if value="${sim_ignition != ''}"> <xacro:property name="_sim_ignition" value="${sim_ignition}" lazy_eval="false"/> </xacro:if>
+    <xacro:if value="${port != ''}"> <xacro:property name="_port" value="${port}" lazy_eval="false"/> </xacro:if>
+    <xacro:if value="${baud != ''}"> <xacro:property name="_baud" value="${baud}" lazy_eval="false"/> </xacro:if>
+    <xacro:if value="${timeout != ''}"> <xacro:property name="_timeout" value="${timeout}" lazy_eval="false"/> </xacro:if>
+    <xacro:if value="${conversion != ''}"> <xacro:property name="_conversion" value="${conversion}" lazy_eval="false"/> </xacro:if>
+    <xacro:if value="${rated_effort != ''}"> <xacro:property name="_rated_effort" value="${rated_effort}" lazy_eval="false"/> </xacro:if>
+    <xacro:if value="${tolerance != ''}"> <xacro:property name="_tolerance" value="${tolerance}" lazy_eval="false"/> </xacro:if>
     <!-- Ewellix Description -->
     <xacro:ewellix_lift
@@ -45,4 +64,10 @@
       use_fake_hardware="${_use_fake_hardware}"
       sim_ignition="${_sim_ignition}"
+      port="${_port}"
+      baud="${_baud}"
+      timeout="${_timeout}"
+      conversion="${_conversion}"
+      rated_effort="${_rated_effort}"
+      tolerance="${_tolerance}"
       >
       <xacro:insert_block name="origin"/>
